Commit message: 11less

File: description/lidar.xacro (robot description, xacro)
@@ -22,3 +22,33 @@
         </xacro:inertial_cylinder>
     </link>
+    <gazebo reference="laser_frame">
+        <material>Gazebo/Red</material>
+        <!-- Добавим симуляцию сенсора. Тип указывает на сканирующий лидар -->
+        <sensor name="laser" type="ray">
+            <pose> 0 0 0 0 0 0 </pose>
+            <visualize>false</visualize>
+            <update_rate>10</update_rate>
+            <ray>
+                <scan>
+                    <horizontal>
+                        <samples>360</samples>
+                        <min_angle>-3.14</min_angle>
+                        <max_angle>3.14</max_angle>
+                    </horizontal>
+                </scan>
+                <range>
+                    <min>0.3</min>
+                    <max>12</max>
+                </range>
+            </ray>
+            <!-- Добавим плагин для общения рос и газебо -->
+            <plugin name="laser_controller" filename="libgazebo_ros_ray_sensor.so">
+                <ros>
+                    <argument>~/out:=scan</argument>
+                </ros>
+                <output_type>sensor_msgs/LaserScan</output_type>
+                <frame_name>laser_frame</frame_name>
+            </plugin>
+        </sensor>
+    </gazebo>
 </robot>

File: description/robot.urdf.xacro (robot description, xacro)
@@ -8,3 +8,5 @@
     <!-- Включаем описание лидара -->
     <xacro:include filename="lidar.xacro"/>
+    <!-- Включаем описание камеры -->
+    <xacro:include filename="camera.xacro"/>
 </robot>
