Commit message: less2

File: description/robot.urdf.xacro (robot description, xacro)
@@ -3,4 +3,4 @@
     <!-- Вкладка "робот" со строкой сверху - это стандартное описание xacro файла -->
     <!-- Стандартный вид ссылки -->
-    <link name="base_link"></link>
+    <xacro:include filename="robot_core.xacro"/>
 </robot>

Commit message: 8less

File: description/robot.urdf.xacro (robot description, xacro)
@@ -6,3 +6,5 @@
     <!-- Включаем описание взаимодействия робота и Gazebo -->
     <xacro:include filename="gazebo_control.xacro"/>
+    <!-- Включаем описание лидара -->
+    <xacro:include filename="lidar.xacro"/>
 </robot>

File: description/robot_core.xacro (robot description, xacro)
@@ -14,4 +14,7 @@
 <material name="black">
     <color rgba="0 0 0 1"/>
+</material>
+<material name="red">
+    <color rgba="1 0 0 1"/>
 </material>
 <!-- Базовая ссылка -->

Commit message: 14less

File: description/robot.urdf.xacro (robot description, xacro)
@@ -2,11 +2,21 @@
 <robot xmlns:xacro="http://www.ros.org/wiki/xacro"  name="robot">
     <!-- Вкладка "робот" со строкой сверху - это стандартное описание xacro файла -->
+    <xacro:arg name="use_ros2_control" default="true"/>
     <!-- Включаем описание робота -->
     <xacro:include filename="robot_core.xacro"/>
+    <!-- <xacro:include filename="ros2_control.xacro"/> -->
+    <xacro:if value="$(arg use_ros2_control)">
+        <xacro:include filename="ros2_control.xacro"/>
+    </xacro:if>
+    <xacro:unless value="$(arg use_ros2_control)">
+        <xacro:include filename="gazebo_control.xacro"/>
+    </xacro:unless>
     <!-- Включаем описание взаимодействия робота и Gazebo -->
-    <xacro:include filename="gazebo_control.xacro"/>
+    <!-- <xacro:include filename="gazebo_control.xacro"/> -->
     <!-- Включаем описание лидара -->
     <xacro:include filename="lidar.xacro"/>
     <!-- Включаем описание камеры -->
     <xacro:include filename="camera.xacro"/>
+    <!-- Включаем описание взаимодействия робота и ros2_control -->
+    <!-- <xacro:include filename="ros2_control.xacro"/> -->
 </robot>

File: description/robot_core.xacro (robot description, xacro)
@@ -64,5 +64,5 @@
     <collision>
         <geometry>
-            <cylinder radius="0.05" length="0.04"/>
+            <sphere radius="0.05"/>
         </geometry>
     </collision>
@@ -90,5 +90,5 @@
     <collision>
         <geometry>
-            <cylinder radius="0.05" length="0.04"/>
+            <sphere radius="0.05"/>
         </geometry>
     </collision>
